File: PCB/DVDLaserScannerII/DVDLaserScanner.sch (KiCad schematic (older format))
At the start: 78 parts, among them Q1 Q_NMOS_GDS, SW1 BUT, U1 MCP4922-E/SL, U10 Con45, U11 Con45, U12 Con45, U13 TLC2274, U2 MCP4922-E/SL, U3 ARDUINO_MICRO, U4 TCA0372_DWG, U5 TCA0372_DWG, U6 TCA0372_DWG, U7 MCP6002, U8 MCP4922-E/SL, U9 TLC2274, X1 MountPad3, X2 MountPad3, X3 MountPad3, X4 MountPad3, X5 PAD, X6 PAD, X7 PAD

Commit message: Updated Schematic PDF
Parts:
- R14, R19: value 470 -> 560
- R23, R31: value 180k -> 220k
Changed lines of the file:
@@
 U 1 1 586F2910
 P 13150 8000
-F 0 "R13" V 13265 8000 50  0000 C CNN
+F 0 "R13" H 13265 8000 50  0000 C CNN
 F 1 "3.3k" V 13356 8000 50  0000 C CNN
 F 2 "GaudiLabsFootPrints:0805G" V 13080 8000 50  0001 C CNN
@@
 P 3650 9000
 F 0 "R19" V 3765 9000 50  0000 C CNN
-F 1 "470" V 3856 9000 50  0000 C CNN
+F 1 "560" V 3856 9000 50  0000 C CNN
 F 2 "GaudiLabsFootPrints:0805G" V 3580 9000 50  0001 C CNN
 F 3 "" H 3650 9000 50  0000 C CNN
@@
 P 1200 6800
 F 0 "R14" V 1315 6800 50  0000 C CNN
-F 1 "470" V 1406 6800 50  0000 C CNN
+F 1 "560" V 1406 6800 50  0000 C CNN
 F 2 "GaudiLabsFootPrints:0805G" V 1130 6800 50  0001 C CNN
 F 3 "" H 1200 6800 50  0000 C CNN
@@
 U 1 1 592943E8
 P 4150 9400
-F 0 "C7" H 3900 9450 50  0000 L CNN
-F 1 "100n" H 4200 9150 50  0000 L CNN
+F 0 "C7" H 4000 9300 50  0000 L CNN
+F 1 "100n" H 3950 9550 50  0000 L CNN
 F 2 "GaudiLabsFootPrints:0805G" H 4150 9400 50  0001 C CNN
 F 3 "" H 4150 9400 50  0000 C CNN
@@
 P 7750 3800
 F 0 "R23" V 7600 3550 50  0000 L CNN
-F 1 "180k" V 7650 3700 50  0000 L CNN
+F 1 "220k" V 7650 3700 50  0000 L CNN
 F 2 "GaudiLabsFootPrints:0805G" V 7680 3800 50  0001 C CNN
 F 3 "" H 7750 3800 50  0000 C CNN
@@
 P 7750 5300
 F 0 "R31" V 7650 5100 50  0000 L CNN
-F 1 "180k" V 7650 5200 50  0000 L CNN
+F 1 "220k" V 7650 5300 50  0000 L CNN
 F 2 "GaudiLabsFootPrints:0805G" V 7680 5300 50  0001 C CNN
 F 3 "" H 7750 5300 50  0000 C CNN
@@
 U 1 1 592C0CA6
 P 4350 9400
-F 0 "C6" H 4100 9450 50  0000 L CNN
+F 0 "C6" H 4400 9300 50  0000 L CNN
 F 1 "100n" H 4450 9550 50  0000 L CNN
 F 2 "GaudiLabsFootPrints:0805G" H 4350 9400 50  0001 C CNN
